File: hardware/Kicad/bluetooth_audio/bluetooth_audio.sch (KiCad schematic (older format))
At the start: 4 parts

Commit message: Kicad proj added
Таки добавил проект в KICAD  для обычательных целей.
Parts:
- added J?: AVR-ISP-6, symbol Connector:AVR-ISP-6
- added J?: Conn_01x03, symbol Connector_Generic:Conn_01x03
- added M?: TPA6112_M, symbol Project_lib:TPA6112_M
- added R? (x8): 10K, symbol Device:R
- added R? (x8): 20K, symbol Device:R
- R? (x2): value R -> 200
Connections:
- net labels added: +3V3, +5V, BR_RST, BT_RST, BT_RX, BT_TX, MUTE, NXT, PP, PRV, PWR, V+, V-
- wire segments 8 -> 99
- no-connect marks 0 -> 29
