File: hardware/Kicad/bluetooth_audio/bluetooth_audio.kicad_pcb (KiCad board)
At the start: 0 parts

Commit message: Kicad project started
Parts:
- added U1: ATmega8A-AU, Package_QFP:TQFP-32_7x7mm_P0.8mm, F.Cu at (151.1, 101.6)
Other:
- board outline added: 38.1 x 25.4 mm
- copper layers 0 -> 2
- net class Default added: clearance 0.2, trace_width 0.25, via_dia 0.8, via_drill 0.4
